Commit message: tp add rgb camera

File: install/arduinobot_description/share/arduinobot_description/urdf/arduinobot.urdf.xacro (robot description, xacro)
@@ -107,3 +107,18 @@
         <limit lower="0.0" upper="${PI/2}" effort="${effort}" velocity="${velocity}" />
     </joint>
+    <link name="rgb_camera">
+        <visual>
+            <origin rpy="0 -0.5 1.57" xyz="0 0.45 0.2" />
+            <geometry>
+                <mesh filename="package://arduinobot_description/meshes/pi_camera.STL" scale="0.01 0.01 0.01" />
+            </geometry>
+        </visual>
+    </link>
+    <joint name="rgb_camera_joint" type="revolute">
+        <parent link="base_link" />
+        <child link="rgb_camera"  />
+        <origin rpy="0 -${PI/6} ${PI/2}" xyz="0 0.45 0.2" />
+        <axis xyz="0 0 1"/>
+        <limit lower="0.0" upper="${PI/2}" effort="${effort}" velocity="${velocity}" />
+    </joint>
 </robot>

File: src/arduinobot_description/urdf/arduinobot.urdf.xacro (robot description, xacro)
@@ -86,5 +86,5 @@
     <link name="gripper_left">
         <visual>
-            <origin rpy="0 0 -${PI/2}" xyz="-0.04 0.5 -0.1" />  <!-- la position de l'origine dans le visual-->
+            <origin rpy="0 0 -${PI/2}" xyz="-0.04 0.5 -0.1" />  <!-- la position du STL par rapport à son repère link-->
             <geometry>
                 <mesh filename="package://arduinobot_description/meshes/left_finger.STL" scale="0.01 0.01 0.01" />
@@ -107,3 +107,20 @@
         <limit lower="0.0" upper="${PI/2}" effort="${effort}" velocity="${velocity}" />
     </joint>
+    <link name="rgb_camera">
+        <visual>
+            <!--origin rpy="0 ${PI/2} 0" xyz="-0.05 -0.14 0.12" /-->
+            <origin rpy="-1.57 0 -1.57" xyz="-0.1 0.125 0.15"/>
+            <geometry>
+                <mesh filename="package://arduinobot_description/meshes/pi_camera.STL" scale="0.01 0.01 0.01" />
+            </geometry>
+        </visual>
+    </link>
+    <joint name="rgb_camera_joint" type="fixed">
+        <parent link="base_link" />
+        <child link="rgb_camera"  />
+        <!--origin rpy="0 -${PI/6} ${PI/2}" xyz="0 0.45 0.2" /-->
+        <origin rpy="0 -0.5 1.57" xyz="0 0.4 0.2" />  <!-- la position du STL par rapport à son repère link-->
+        <axis xyz="0 0 1"/>
+        <limit lower="-${PI/2}" upper="${PI/2}" effort="${effort}" velocity="${velocity}" />
+    </joint>
 </robot>

Commit message: clavier

File: install/arduinobot_description/share/arduinobot_description/urdf/arduinobot.urdf.xacro (robot description, xacro)
@@ -4,6 +4,15 @@
     <xacro:property name="effort" value="30.0" />
     <xacro:property name="velocity" value="10.0" />
+    <xacro:macro name="default_inertia" params="mass">
+        <inertia>
+            <mass value="${mass}" />
+            <inertia ixx="1.0" ixy="0.0" ixz="0.0"
+                    iyy="1.0" iyz="0.0"
+                    izz="1.0" />
+        </inertia>
+    </xacro:macro>
     <link name="world" />
     <link name="base_link">
+        <xacro:default_inertia  mass="1.0" />
         <visual>
             <origin rpy="0 0 0" xyz="-0.5 -0.5 0" />
@@ -12,4 +21,10 @@
             </geometry>
         </visual>
+        <collision>
+            <origin rpy="0 0 0" xyz="-0.5 -0.5 0" />
+            <geometry>
+                <mesh filename="package://arduinobot_description/meshes/basement.STL" scale="0.01 0.01 0.01" />
+            </geometry>
+        </collision>
     </link>
     <joint name="virtual_join" type="fixed">
@@ -19,4 +34,5 @@
     </joint>
     <link name="base_plate">
+        <xacro:default_inertia  mass="1.0" />
         <visual>
             <origin rpy="0 0 0" xyz="-0.39 -0.39 -0.56" />
@@ -25,4 +41,10 @@
             </geometry>
         </visual>
+        <collision>
+            <origin rpy="0 0 0" xyz="-0.39 -0.39 -0.56" />
+            <geometry>
+                <mesh filename="package://arduinobot_description/meshes/base_plate.STL" scale="0.01 0.01 0.01" />
+            </geometry>
+        </collision>
     </link>
     <joint name="joint_1" type="revolute">
@@ -34,4 +56,5 @@
     </joint>
     <link name="forward_drive_arm">
+        <xacro:default_inertia  mass="0.1" />
         <visual>
             <origin rpy="0 -${PI/2} ${PI/2}" xyz="0.19 0.06 -0.06" />
@@ -40,4 +63,10 @@
             </geometry>
         </visual>
+        <collision>
+            <origin rpy="0 -${PI/2} ${PI/2}" xyz="0.19 0.06 -0.06" />
+            <geometry>
+                <mesh filename="package://arduinobot_description/meshes/forward_drive_arm.STL" scale="0.01 0.01 0.01" />
+            </geometry>
+        </collision>
     </link>
     <joint name="joint_2" type="revolute">
@@ -49,4 +78,5 @@
     </joint>
     <link name="horizontal_arm">
+        <xacro:default_inertia  mass="0.1" />
         <visual>
             <origin rpy="${PI/2} 0 ${PI/2}" xyz="-0.03 -0.4 -0.06" />  <!-- la position de l'origine dans le visual-->
@@ -55,4 +85,10 @@
             </geometry>
         </visual>
+        <collision>
+            <origin rpy="${PI/2} 0 ${PI/2}" xyz="-0.03 -0.4 -0.06" />  <!-- la position de l'origine dans le visual-->
+            <geometry>
+                <mesh filename="package://arduinobot_description/meshes/horizontal_arm.STL" scale="0.01 0.01 0.01" />
+            </geometry>
+        </collision>
     </link>
     <joint name="joint_3" type="revolute">
@@ -64,4 +100,5 @@
     </joint>
     <link name="claw_support">
+        <xacro:default_inertia  mass="0.05" />
         <visual>
             <origin rpy="0 0 ${PI/2}" xyz="0 -0.05 -0.15" />  <!-- la position de l'origine dans le visual-->
@@ -70,4 +107,10 @@
             </geometry>
         </visual>
+        <collision>
+            <origin rpy="0 0 ${PI/2}" xyz="0 -0.05 -0.15" />  <!-- la position de l'origine dans le visual-->
+            <geometry>
+                <mesh filename="package://arduinobot_description/meshes/claw_support.STL" scale="0.01 0.01 0.01" />
+            </geometry>
+        </collision>
     </link>
     <joint name="horizontal_arm_to_claw_support" type="fixed">
@@ -77,4 +120,5 @@
     </joint>
     <link name="gripper_right">
+        <xacro:default_inertia  mass="0.01" />
         <visual>
             <origin rpy="0 0 -${PI/2}" xyz="-0.1 0.5 -0.1" />  <!-- la position de l'origine dans le visual-->
@@ -83,12 +127,25 @@
             </geometry>
         </visual>
+        <collision>
+            <origin rpy="0 0 -${PI/2}" xyz="-0.1 0.5 -0.1" />  <!-- la position de l'origine dans le visual-->
+            <geometry>
+                <mesh filename="package://arduinobot_description/meshes/right_finger.STL" scale="0.01 0.01 0.01" />
+            </geometry>
+        </collision>
     </link>
     <link name="gripper_left">
+        <xacro:default_inertia  mass="0.01" />
         <visual>
-            <origin rpy="0 0 -${PI/2}" xyz="-0.04 0.5 -0.1" />  <!-- la position de l'origine dans le visual-->
+            <origin rpy="0 0 -${PI/2}" xyz="-0.04 0.5 -0.1" />  <!-- la position du STL par rapport à son repère link-->
             <geometry>
                 <mesh filename="package://arduinobot_description/meshes/left_finger.STL" scale="0.01 0.01 0.01" />
             </geometry>
         </visual>
+        <collision>
+            <origin rpy="0 0 -${PI/2}" xyz="-0.04 0.5 -0.1" />  <!-- la position du STL par rapport à son repère link-->
+            <geometry>
+                <mesh filename="package://arduinobot_description/meshes/left_finger.STL" scale="0.01 0.01 0.01" />
+            </geometry>
+        </collision>
     </link>
     <joint name="joint_4" type="revolute">
@@ -109,16 +166,24 @@
     <link name="rgb_camera">
         <visual>
-            <origin rpy="0 -0.5 1.57" xyz="0 0.45 0.2" />
+            <!--origin rpy="0 ${PI/2} 0" xyz="-0.05 -0.14 0.12" /-->
+            <origin rpy="-1.57 0 -1.57" xyz="-0.1 0.125 0.15"/>
             <geometry>
                 <mesh filename="package://arduinobot_description/meshes/pi_camera.STL" scale="0.01 0.01 0.01" />
             </geometry>
         </visual>
+        <collision>
+            <origin rpy="-1.57 0 -1.57" xyz="-0.1 0.125 0.15"/>
+            <geometry>
+                <mesh filename="package://arduinobot_description/meshes/pi_camera.STL" scale="0.01 0.01 0.01" />
+            </geometry>
+        </collision>
     </link>
-    <joint name="rgb_camera_joint" type="revolute">
+    <joint name="rgb_camera_joint" type="fixed">
         <parent link="base_link" />
         <child link="rgb_camera"  />
-        <origin rpy="0 -${PI/6} ${PI/2}" xyz="0 0.45 0.2" />
+        <!--origin rpy="0 -${PI/6} ${PI/2}" xyz="0 0.45 0.2" /-->
+        <origin rpy="0 -0.5 1.57" xyz="0 0.4 0.2" />  <!-- la position du STL par rapport à son repère link-->
         <axis xyz="0 0 1"/>
-        <limit lower="0.0" upper="${PI/2}" effort="${effort}" velocity="${velocity}" />
+        <limit lower="-${PI/2}" upper="${PI/2}" effort="${effort}" velocity="${velocity}" />
     </joint>
 </robot>

File: src/arduinobot_description/urdf/arduinobot.urdf.xacro (robot description, xacro)
@@ -4,6 +4,15 @@
     <xacro:property name="effort" value="30.0" />
     <xacro:property name="velocity" value="10.0" />
+    <xacro:macro name="default_inertia" params="mass">
+        <inertia>
+            <mass value="${mass}" />
+            <inertia ixx="1.0" ixy="0.0" ixz="0.0"
+                    iyy="1.0" iyz="0.0"
+                    izz="1.0" />
+        </inertia>
+    </xacro:macro>
     <link name="world" />
     <link name="base_link">
+        <xacro:default_inertia  mass="1.0" />
         <visual>
             <origin rpy="0 0 0" xyz="-0.5 -0.5 0" />
@@ -12,4 +21,10 @@
             </geometry>
         </visual>
+        <collision>
+            <origin rpy="0 0 0" xyz="-0.5 -0.5 0" />
+            <geometry>
+                <mesh filename="package://arduinobot_description/meshes/basement.STL" scale="0.01 0.01 0.01" />
+            </geometry>
+        </collision>
     </link>
     <joint name="virtual_join" type="fixed">
@@ -19,4 +34,5 @@
     </joint>
     <link name="base_plate">
+        <xacro:default_inertia  mass="1.0" />
         <visual>
             <origin rpy="0 0 0" xyz="-0.39 -0.39 -0.56" />
@@ -25,4 +41,10 @@
             </geometry>
         </visual>
+        <collision>
+            <origin rpy="0 0 0" xyz="-0.39 -0.39 -0.56" />
+            <geometry>
+                <mesh filename="package://arduinobot_description/meshes/base_plate.STL" scale="0.01 0.01 0.01" />
+            </geometry>
+        </collision>
     </link>
     <joint name="joint_1" type="revolute">
@@ -34,4 +56,5 @@
     </joint>
     <link name="forward_drive_arm">
+        <xacro:default_inertia  mass="0.1" />
         <visual>
             <origin rpy="0 -${PI/2} ${PI/2}" xyz="0.19 0.06 -0.06" />
@@ -40,4 +63,10 @@
             </geometry>
         </visual>
+        <collision>
+            <origin rpy="0 -${PI/2} ${PI/2}" xyz="0.19 0.06 -0.06" />
+            <geometry>
+                <mesh filename="package://arduinobot_description/meshes/forward_drive_arm.STL" scale="0.01 0.01 0.01" />
+            </geometry>
+        </collision>
     </link>
     <joint name="joint_2" type="revolute">
@@ -49,4 +78,5 @@
     </joint>
     <link name="horizontal_arm">
+        <xacro:default_inertia  mass="0.1" />
         <visual>
             <origin rpy="${PI/2} 0 ${PI/2}" xyz="-0.03 -0.4 -0.06" />  <!-- la position de l'origine dans le visual-->
@@ -55,4 +85,10 @@
             </geometry>
         </visual>
+        <collision>
+            <origin rpy="${PI/2} 0 ${PI/2}" xyz="-0.03 -0.4 -0.06" />  <!-- la position de l'origine dans le visual-->
+            <geometry>
+                <mesh filename="package://arduinobot_description/meshes/horizontal_arm.STL" scale="0.01 0.01 0.01" />
+            </geometry>
+        </collision>
     </link>
     <joint name="joint_3" type="revolute">
@@ -64,4 +100,5 @@
     </joint>
     <link name="claw_support">
+        <xacro:default_inertia  mass="0.05" />
         <visual>
             <origin rpy="0 0 ${PI/2}" xyz="0 -0.05 -0.15" />  <!-- la position de l'origine dans le visual-->
@@ -70,4 +107,10 @@
             </geometry>
         </visual>
+        <collision>
+            <origin rpy="0 0 ${PI/2}" xyz="0 -0.05 -0.15" />  <!-- la position de l'origine dans le visual-->
+            <geometry>
+                <mesh filename="package://arduinobot_description/meshes/claw_support.STL" scale="0.01 0.01 0.01" />
+            </geometry>
+        </collision>
     </link>
     <joint name="horizontal_arm_to_claw_support" type="fixed">
@@ -77,4 +120,5 @@
     </joint>
     <link name="gripper_right">
+        <xacro:default_inertia  mass="0.01" />
         <visual>
             <origin rpy="0 0 -${PI/2}" xyz="-0.1 0.5 -0.1" />  <!-- la position de l'origine dans le visual-->
@@ -83,6 +127,13 @@
             </geometry>
         </visual>
+        <collision>
+            <origin rpy="0 0 -${PI/2}" xyz="-0.1 0.5 -0.1" />  <!-- la position de l'origine dans le visual-->
+            <geometry>
+                <mesh filename="package://arduinobot_description/meshes/right_finger.STL" scale="0.01 0.01 0.01" />
+            </geometry>
+        </collision>
     </link>
     <link name="gripper_left">
+        <xacro:default_inertia  mass="0.01" />
         <visual>
             <origin rpy="0 0 -${PI/2}" xyz="-0.04 0.5 -0.1" />  <!-- la position du STL par rapport à son repère link-->
@@ -91,4 +142,10 @@
             </geometry>
         </visual>
+        <collision>
+            <origin rpy="0 0 -${PI/2}" xyz="-0.04 0.5 -0.1" />  <!-- la position du STL par rapport à son repère link-->
+            <geometry>
+                <mesh filename="package://arduinobot_description/meshes/left_finger.STL" scale="0.01 0.01 0.01" />
+            </geometry>
+        </collision>
     </link>
     <joint name="joint_4" type="revolute">
@@ -115,4 +172,10 @@
             </geometry>
         </visual>
+        <collision>
+            <origin rpy="-1.57 0 -1.57" xyz="-0.1 0.125 0.15"/>
+            <geometry>
+                <mesh filename="package://arduinobot_description/meshes/pi_camera.STL" scale="0.01 0.01 0.01" />
+            </geometry>
+        </collision>
     </link>
     <joint name="rgb_camera_joint" type="fixed">
