Commit message: urdf gazebo ros2 control

File: install/arduinobot_description/share/arduinobot_description/urdf/arduinobot.urdf.xacro (robot description, xacro)
@@ -1,189 +1 @@
-<?xml version="1.0"?>
-<robot xmlns:xacro="http://www.ros.org/wiki/xacro" name="arduinobot">
-    <xacro:property name="PI" value="3.14159" />
-    <xacro:property name="effort" value="30.0" />
-    <xacro:property name="velocity" value="10.0" />
-    <xacro:macro name="default_inertia" params="mass">
-        <inertia>
-            <mass value="${mass}" />
-            <inertia ixx="1.0" ixy="0.0" ixz="0.0"
-                    iyy="1.0" iyz="0.0"
-                    izz="1.0" />
-        </inertia>
-    </xacro:macro>
-    <link name="world" />
-    <link name="base_link">
-        <xacro:default_inertia  mass="1.0" />
-        <visual>
-            <origin rpy="0 0 0" xyz="-0.5 -0.5 0" />
-            <geometry>
-                <mesh filename="package://arduinobot_description/meshes/basement.STL" scale="0.01 0.01 0.01" />
-            </geometry>
-        </visual>
-        <collision>
-            <origin rpy="0 0 0" xyz="-0.5 -0.5 0" />
-            <geometry>
-                <mesh filename="package://arduinobot_description/meshes/basement.STL" scale="0.01 0.01 0.01" />
-            </geometry>
-        </collision>
-    </link>
-    <joint name="virtual_join" type="fixed">
-        <parent link="world"/>
-        <child link="base_link"/>
-        <origin rpy="0 0 0" xyz="0 0 0" />
-    </joint>
-    <link name="base_plate">
-        <xacro:default_inertia  mass="1.0" />
-        <visual>
-            <origin rpy="0 0 0" xyz="-0.39 -0.39 -0.56" />
-            <geometry>
-                <mesh filename="package://arduinobot_description/meshes/base_plate.STL" scale="0.01 0.01 0.01" />
-            </geometry>
-        </visual>
-        <collision>
-            <origin rpy="0 0 0" xyz="-0.39 -0.39 -0.56" />
-            <geometry>
-                <mesh filename="package://arduinobot_description/meshes/base_plate.STL" scale="0.01 0.01 0.01" />
-            </geometry>
-        </collision>
-    </link>
-    <joint name="joint_1" type="revolute">
-        <parent link="base_link"/>
-        <child link="base_plate"/>
-        <axis xyz="0 0 1" /> <!--va roter (le revolute, rotoide !=fixed) autour de l'axe z-->
-        <origin rpy="0 0 0" xyz="0 0 0.307" /> <!-- orientation du repère child par rapport au repère parent  -->
-        <limit lower="-${PI/2}" upper="${PI/2}" effort="${effort}" velocity="${velocity}" />
-    </joint>
-    <link name="forward_drive_arm">
-        <xacro:default_inertia  mass="0.1" />
-        <visual>
-            <origin rpy="0 -${PI/2} ${PI/2}" xyz="0.19 0.06 -0.06" />
-            <geometry>
-                <mesh filename="package://arduinobot_description/meshes/forward_drive_arm.STL" scale="0.01 0.01 0.01" />
-            </geometry>
-        </visual>
-        <collision>
-            <origin rpy="0 -${PI/2} ${PI/2}" xyz="0.19 0.06 -0.06" />
-            <geometry>
-                <mesh filename="package://arduinobot_description/meshes/forward_drive_arm.STL" scale="0.01 0.01 0.01" />
-            </geometry>
-        </collision>
-    </link>
-    <joint name="joint_2" type="revolute">
-        <parent link="base_plate"/>
-        <child link="forward_drive_arm"/>
-        <axis xyz="0 0 1" /> <!--va roter (le revolute, rotoide !=fixed) autour de l'axe z -->
-        <origin rpy="0 0 0" xyz="-0.02 0 0.35" /> <!-- orientation du repère child par rapport au repère parent -->
-        <limit lower="-${PI/2}" upper="${PI/2}" effort="${effort}" velocity="${velocity}" />
-    </joint>
-    <link name="horizontal_arm">
-        <xacro:default_inertia  mass="0.1" />
-        <visual>
-            <origin rpy="${PI/2} 0 ${PI/2}" xyz="-0.03 -0.4 -0.06" />  <!-- la position de l'origine dans le visual-->
-            <geometry>
-                <mesh filename="package://arduinobot_description/meshes/horizontal_arm.STL" scale="0.01 0.01 0.01" />
-            </geometry>
-        </visual>
-        <collision>
-            <origin rpy="${PI/2} 0 ${PI/2}" xyz="-0.03 -0.4 -0.06" />  <!-- la position de l'origine dans le visual-->
-            <geometry>
-                <mesh filename="package://arduinobot_description/meshes/horizontal_arm.STL" scale="0.01 0.01 0.01" />
-            </geometry>
-        </collision>
-    </link>
-    <joint name="joint_3" type="revolute">
-        <parent link="forward_drive_arm"/>
-        <child link="horizontal_arm"/>
-        <axis xyz="1 0 0" /> <!--va roter (le revolute, rotoide !=fixed) autour de l'axe z -->
-        <origin rpy="0 0 0" xyz="0 0 0.8" /> <!-- orientation du repère child par rapport au repère parent -->
-        <limit lower="-${PI/2}" upper="${PI/2}" effort="${effort}" velocity="${velocity}" />
-    </joint>
-    <link name="claw_support">
-        <xacro:default_inertia  mass="0.05" />
-        <visual>
-            <origin rpy="0 0 ${PI/2}" xyz="0 -0.05 -0.15" />  <!-- la position de l'origine dans le visual-->
-            <geometry>
-                <mesh filename="package://arduinobot_description/meshes/claw_support.STL" scale="0.01 0.01 0.01" />
-            </geometry>
-        </visual>
-        <collision>
-            <origin rpy="0 0 ${PI/2}" xyz="0 -0.05 -0.15" />  <!-- la position de l'origine dans le visual-->
-            <geometry>
-                <mesh filename="package://arduinobot_description/meshes/claw_support.STL" scale="0.01 0.01 0.01" />
-            </geometry>
-        </collision>
-    </link>
-    <joint name="horizontal_arm_to_claw_support" type="fixed">
-        <parent link="horizontal_arm"/>
-        <child link="claw_support"/>
-        <origin rpy="0 0 0" xyz="0 0.82 0" /> <!-- orientation du repère child par rapport au repère parent -->
-    </joint>
-    <link name="gripper_right">
-        <xacro:default_inertia  mass="0.01" />
-        <visual>
-            <origin rpy="0 0 -${PI/2}" xyz="-0.1 0.5 -0.1" />  <!-- la position de l'origine dans le visual-->
-            <geometry>
-                <mesh filename="package://arduinobot_description/meshes/right_finger.STL" scale="0.01 0.01 0.01" />
-            </geometry>
-        </visual>
-        <collision>
-            <origin rpy="0 0 -${PI/2}" xyz="-0.1 0.5 -0.1" />  <!-- la position de l'origine dans le visual-->
-            <geometry>
-                <mesh filename="package://arduinobot_description/meshes/right_finger.STL" scale="0.01 0.01 0.01" />
-            </geometry>
-        </collision>
-    </link>
-    <link name="gripper_left">
-        <xacro:default_inertia  mass="0.01" />
-        <visual>
-            <origin rpy="0 0 -${PI/2}" xyz="-0.04 0.5 -0.1" />  <!-- la position du STL par rapport à son repère link-->
-            <geometry>
-                <mesh filename="package://arduinobot_description/meshes/left_finger.STL" scale="0.01 0.01 0.01" />
-            </geometry>
-        </visual>
-        <collision>
-            <origin rpy="0 0 -${PI/2}" xyz="-0.04 0.5 -0.1" />  <!-- la position du STL par rapport à son repère link-->
-            <geometry>
-                <mesh filename="package://arduinobot_description/meshes/left_finger.STL" scale="0.01 0.01 0.01" />
-            </geometry>
-        </collision>
-    </link>
-    <joint name="joint_4" type="revolute">
-        <parent link="claw_support"/>
-        <child link="gripper_right"/>
-        <axis xyz="0 0 1"/>
-        <origin rpy="0 0 0" xyz="-0.04 0.13 -0.1" /> <!-- orientation du repère child par rapport au repère parent -->
-        <limit lower="-${PI/2}" upper="0.0" effort="${effort}" velocity="${velocity}" />
-    </joint>
-    <joint name="joint_5" type="revolute">
-        <parent link="claw_support"/>
-        <child link="gripper_left"/>
-        <axis xyz="0 0 1"/>
-        <origin rpy="0 0 0" xyz="-0.22 0.13 -0.1" /> <!-- orientation du repère child par rapport au repère parent -->
-        <mimic joint="joint_4" multiplier="-1" />
-        <limit lower="0.0" upper="${PI/2}" effort="${effort}" velocity="${velocity}" />
-    </joint>
-    <link name="rgb_camera">
-        <visual>
-            <!--origin rpy="0 ${PI/2} 0" xyz="-0.05 -0.14 0.12" /-->
-            <origin rpy="-1.57 0 -1.57" xyz="-0.1 0.125 0.15"/>
-            <geometry>
-                <mesh filename="package://arduinobot_description/meshes/pi_camera.STL" scale="0.01 0.01 0.01" />
-            </geometry>
-        </visual>
-        <collision>
-            <origin rpy="-1.57 0 -1.57" xyz="-0.1 0.125 0.15"/>
-            <geometry>
-                <mesh filename="package://arduinobot_description/meshes/pi_camera.STL" scale="0.01 0.01 0.01" />
-            </geometry>
-        </collision>
-    </link>
-    <joint name="rgb_camera_joint" type="fixed">
-        <parent link="base_link" />
-        <child link="rgb_camera"  />
-        <!--origin rpy="0 -${PI/6} ${PI/2}" xyz="0 0.45 0.2" /-->
-        <origin rpy="0 -0.5 1.57" xyz="0 0.4 0.2" />  <!-- la position du STL par rapport à son repère link-->
-        <axis xyz="0 0 1"/>
-        <limit lower="-${PI/2}" upper="${PI/2}" effort="${effort}" velocity="${velocity}" />
-    </joint>
-</robot>
+/home/marcos/arduinobot_ws/src/arduinobot_description/urdf/arduinobot.urdf.xacro

File: src/arduinobot_description/urdf/arduinobot.urdf.xacro (robot description, xacro)
@@ -1,18 +1,30 @@
 <?xml version="1.0"?>
 <robot xmlns:xacro="http://www.ros.org/wiki/xacro" name="arduinobot">
+    <xacro:include filename="$(find arduinobot_description)/urdf/arduinobot_gazebo.xacro" />
+    <xacro:include filename="$(find arduinobot_description)/urdf/arduinobot_ros2_control.xacro" />
     <xacro:property name="PI" value="3.14159" />
     <xacro:property name="effort" value="30.0" />
     <xacro:property name="velocity" value="10.0" />
-    <xacro:macro name="default_inertia" params="mass">
-        <inertia>
+    <xacro:macro name="default_inertial" params="mass">
+        <inertial>
             <mass value="${mass}" />
             <inertia ixx="1.0" ixy="0.0" ixz="0.0"
                     iyy="1.0" iyz="0.0"
                     izz="1.0" />
-        </inertia>
+        </inertial>
+    </xacro:macro>
+    <xacro:macro name="default_transmission" params="number">
+        <transmission name="transmission_${number}">
+            <plugin>transmission_interface/SimpleTransmission</plugin>
+            <actuator name="motor_${number}" role="actuator1"/>
+            <joint name="joint_${number}" role="joint1">
+                <!-- 1 deg of rotation of the motor correspond to 1 deg of rotation of the joint -->
+                <mechanical_reduction>1.0</mechanical_reduction>
+            </joint>
+        </transmission>
     </xacro:macro>
     <link name="world" />
     <link name="base_link">
-        <xacro:default_inertia  mass="1.0" />
+        <xacro:default_inertial  mass="1.0" />
         <visual>
             <origin rpy="0 0 0" xyz="-0.5 -0.5 0" />
@@ -34,5 +46,5 @@
     </joint>
     <link name="base_plate">
-        <xacro:default_inertia  mass="1.0" />
+        <xacro:default_inertial  mass="1.0" />
         <visual>
             <origin rpy="0 0 0" xyz="-0.39 -0.39 -0.56" />
@@ -56,5 +68,5 @@
     </joint>
     <link name="forward_drive_arm">
-        <xacro:default_inertia  mass="0.1" />
+        <xacro:default_inertial  mass="0.1" />
         <visual>
             <origin rpy="0 -${PI/2} ${PI/2}" xyz="0.19 0.06 -0.06" />
@@ -78,5 +90,5 @@
     </joint>
     <link name="horizontal_arm">
-        <xacro:default_inertia  mass="0.1" />
+        <xacro:default_inertial  mass="0.1" />
         <visual>
             <origin rpy="${PI/2} 0 ${PI/2}" xyz="-0.03 -0.4 -0.06" />  <!-- la position de l'origine dans le visual-->
@@ -100,5 +112,5 @@
     </joint>
     <link name="claw_support">
-        <xacro:default_inertia  mass="0.05" />
+        <xacro:default_inertial  mass="0.05" />
         <visual>
             <origin rpy="0 0 ${PI/2}" xyz="0 -0.05 -0.15" />  <!-- la position de l'origine dans le visual-->
@@ -120,5 +132,5 @@
     </joint>
     <link name="gripper_right">
-        <xacro:default_inertia  mass="0.01" />
+        <xacro:default_inertial  mass="0.01" />
         <visual>
             <origin rpy="0 0 -${PI/2}" xyz="-0.1 0.5 -0.1" />  <!-- la position de l'origine dans le visual-->
@@ -135,5 +147,5 @@
     </link>
     <link name="gripper_left">
-        <xacro:default_inertia  mass="0.01" />
+        <xacro:default_inertial  mass="0.01" />
         <visual>
             <origin rpy="0 0 -${PI/2}" xyz="-0.04 0.5 -0.1" />  <!-- la position du STL par rapport à son repère link-->
@@ -165,6 +177,6 @@
     </joint>
     <link name="rgb_camera">
-        <visual>
-            <!--origin rpy="0 ${PI/2} 0" xyz="-0.05 -0.14 0.12" /-->
+        <xacro:default_inertial  mass="0.001" />
+        <visual>
             <origin rpy="-1.57 0 -1.57" xyz="-0.1 0.125 0.15"/>
             <geometry>
@@ -182,8 +194,47 @@
         <parent link="base_link" />
         <child link="rgb_camera"  />
-        <!--origin rpy="0 -${PI/6} ${PI/2}" xyz="0 0.45 0.2" /-->
-        <origin rpy="0 -0.5 1.57" xyz="0 0.4 0.2" />  <!-- la position du STL par rapport à son repère link-->
+        <origin rpy="0 -0.5 1.57" xyz="0 0.4 0.2" />
         <axis xyz="0 0 1"/>
         <limit lower="-${PI/2}" upper="${PI/2}" effort="${effort}" velocity="${velocity}" />
     </joint>
+    <xacro:default_transmission number="1"/>
+    <xacro:default_transmission number="2"/>
+    <xacro:default_transmission number="3"/>
+    <xacro:default_transmission number="4"/>
+    <!-- -->
+    <gazebo  reference="rgb_camera">
+        <sensor  type="camera" name="rgb_camera">
+            <always_on>0</always_on>
+            <!-- fps -->
+            <update_rate>30.0</update_rate>
+            <camera name="camera_name">
+                <horizontal_fov>1.15</horizontal_fov>
+                <vertical_fov>0.71</vertical_fov>
+                <image>
+                    <width>2304</width>
+                    <height>1296</height>
+                    <format>R8G8B8</format>
+                </image>
+              <distortion>
+                <k1>0.1</k1>
+                <k2>0.2</k2>
+                <k3>0.3</k3>
+                <p1>0.4</p1>
+                <p2>0.5</p2>
+                <center>0.5 0.5</center>
+              </distortion>
+            </camera>
+            <!-- Use camera, not camera_triggered -->
+            <plugin name="plugin_name" filename="libgazebo_ros_camera.so">
+              <ros>
+                <!-- <namespace>custom_ns</namespace> -->
+                <remapping>image_raw:=image_raw</remapping>
+                <remapping>camera_info:=camera_info</remapping>
+              </ros>
+              <camera_name>rgb_camera</camera_name>
+              <frame_name>rgb_camera</frame_name>
+              <hack_baseline>0.2</hack_baseline>
+            </plugin>
+          </sensor>
+    </gazebo>
 </robot>
