Commit message: ros controller yaml

File: src/arduinobot_description/urdf/arduinobot.urdf.xacro (robot description, xacro)
@@ -1,6 +1,4 @@
 <?xml version="1.0"?>
 <robot xmlns:xacro="http://www.ros.org/wiki/xacro" name="arduinobot">
-    <xacro:include filename="$(find arduinobot_description)/urdf/arduinobot_gazebo.xacro" />
-    <xacro:include filename="$(find arduinobot_description)/urdf/arduinobot_ros2_control.xacro" />
     <xacro:property name="PI" value="3.14159" />
     <xacro:property name="effort" value="30.0" />
@@ -14,14 +12,4 @@
         </inertial>
     </xacro:macro>
-    <xacro:macro name="default_transmission" params="number">
-        <transmission name="transmission_${number}">
-            <plugin>transmission_interface/SimpleTransmission</plugin>
-            <actuator name="motor_${number}" role="actuator1"/>
-            <joint name="joint_${number}" role="joint1">
-                <!-- 1 deg of rotation of the motor correspond to 1 deg of rotation of the joint -->
-                <mechanical_reduction>1.0</mechanical_reduction>
-            </joint>
-        </transmission>
-    </xacro:macro>
     <link name="world" />
     <link name="base_link">
@@ -198,13 +186,22 @@
         <limit lower="-${PI/2}" upper="${PI/2}" effort="${effort}" velocity="${velocity}" />
     </joint>
-    <xacro:default_transmission number="1"/>
+     <!-- <xacro:include filename="$(find arduinobot_description)/urdf/arduinobot_gazebo.xacro" />
+    <xacro:include filename="$(find arduinobot_description)/urdf/arduinobot_ros2_control.xacro" /> -->
+    <!-- <xacro:macro name="default_transmission" params="number">
+        <transmission name="transmission_${number}">
+            <plugin>transmission_interface/SimpleTransmission</plugin>
+            <actuator name="motor_${number}" role="actuator1"/>
+            <joint name="joint_${number}" role="joint1">
+                <mechanical_reduction>1.0</mechanical_reduction>
+            </joint>
+        </transmission>
+    </xacro:macro> -->
+    <!-- <xacro:default_transmission number="1"/>
     <xacro:default_transmission number="2"/>
     <xacro:default_transmission number="3"/>
     <xacro:default_transmission number="4"/>
-    <!-- -->
     <gazebo  reference="rgb_camera">
         <sensor  type="camera" name="rgb_camera">
             <always_on>0</always_on>
-            <!-- fps -->
             <update_rate>30.0</update_rate>
             <camera name="camera_name">
@@ -225,8 +222,6 @@
               </distortion>
             </camera>
-            <!-- Use camera, not camera_triggered -->
             <plugin name="plugin_name" filename="libgazebo_ros_camera.so">
               <ros>
-                <!-- <namespace>custom_ns</namespace> -->
                 <remapping>image_raw:=image_raw</remapping>
                 <remapping>camera_info:=camera_info</remapping>
@@ -237,4 +232,4 @@
             </plugin>
           </sensor>
-    </gazebo>
+    </gazebo> -->
 </robot>

File: src/arduinobot_description/urdf/arduinobot_gazebo.xacro (robot description, xacro)
@@ -4,6 +4,6 @@
         <plugin filename="libgazebo_ros2_control.so" name="gazebo_ros2_control">
             <robot_param>robot_description</robot_param>
-            <robot_param_node>robot_description</robot_param_node>
-            <params></params>
+            <robot_param_node>robot_state_publisher</robot_param_node>
+            <parameters>$(find arduinobot_controller)/config/arduinobot_controllers.yaml</parameters>
         </plugin>
     </gazebo>

Commit message: service quaternion and euler angles

File: src/arduinobot_description/urdf/arduinobot.urdf.xacro (robot description, xacro)
@@ -1,4 +1,6 @@
 <?xml version="1.0"?>
 <robot xmlns:xacro="http://www.ros.org/wiki/xacro" name="arduinobot">
+    <xacro:include filename="$(find arduinobot_description)/urdf/arduinobot_gazebo.xacro" />
+    <xacro:include filename="$(find arduinobot_description)/urdf/arduinobot_ros2_control.xacro" />
     <xacro:property name="PI" value="3.14159" />
     <xacro:property name="effort" value="30.0" />
@@ -12,4 +14,13 @@
         </inertial>
     </xacro:macro>
+    <xacro:macro name="default_transmission" params="number">
+        <transmission name="transmission_${number}">
+            <plugin>transmission_interface/SimpleTransmission</plugin>
+            <actuator name="motor_${number}" role="actuator1"/>
+            <joint name="joint_${number}" role="joint1">
+                <mechanical_reduction>1.0</mechanical_reduction>
+            </joint>
+        </transmission>
+    </xacro:macro>
     <link name="world" />
     <link name="base_link">
@@ -183,22 +194,10 @@
         <child link="rgb_camera"  />
         <origin rpy="0 -0.5 1.57" xyz="0 0.4 0.2" />
-        <axis xyz="0 0 1"/>
-        <limit lower="-${PI/2}" upper="${PI/2}" effort="${effort}" velocity="${velocity}" />
-    </joint>
-     <!-- <xacro:include filename="$(find arduinobot_description)/urdf/arduinobot_gazebo.xacro" />
-    <xacro:include filename="$(find arduinobot_description)/urdf/arduinobot_ros2_control.xacro" /> -->
-    <!-- <xacro:macro name="default_transmission" params="number">
-        <transmission name="transmission_${number}">
-            <plugin>transmission_interface/SimpleTransmission</plugin>
-            <actuator name="motor_${number}" role="actuator1"/>
-            <joint name="joint_${number}" role="joint1">
-                <mechanical_reduction>1.0</mechanical_reduction>
-            </joint>
-        </transmission>
-    </xacro:macro> -->
-    <!-- <xacro:default_transmission number="1"/>
+    </joint>
+    <xacro:default_transmission number="1"/>
     <xacro:default_transmission number="2"/>
     <xacro:default_transmission number="3"/>
     <xacro:default_transmission number="4"/>
+   <!--
     <gazebo  reference="rgb_camera">
         <sensor  type="camera" name="rgb_camera">
